Commit message: remove comments

File: kaqu_gazebo_sim/description/gazebo_ros2_control_plugin.xacro (robot description, xacro)
@@ -6,6 +6,4 @@
             <plugin>gz_ros2_control/GazeboSimSystem</plugin>
         </hardware>
-        <!-- <xacro:property name="velocity"       value="5"/>
-        <xacro:property name="effort"         value="10"/> 모터 토크 -->
         <joint name="fr_mainbodyhip_joint">
             <command_interface name="position"/>

File: kaqu_gazebo_sim/description/kaqu_joint.xacro (robot description, xacro)
@@ -3,6 +3,6 @@
     <xacro:include filename="$(find kaqu_gazebo_sim)/description/kaqu.gazebo" />
     <xacro:include filename="$(find kaqu_gazebo_sim)/description/kaqu.trans" />
-    <xacro:property name="effort_limit" value="20.0" />
-    <xacro:property name="velocity_limit" value="10.0" />
+    <xacro:property name="effort_limit" value="10.0" />
+    <xacro:property name="velocity_limit" value="3.0" />
     <joint name="fl_mainbodyhip_joint" type="revolute">
         <origin xyz="-0.074 0.077 0.04925" rpy="0 0 0"/>

File: kaqu_gazebo_sim/description/kaqu_link.xacro (robot description, xacro)
@@ -12,11 +12,4 @@
       <inertia ixx="0.00270833" iyy="0.00270" izz="0.00375" ixy="-0.0" iyz="0.0" ixz="0.0"/>
     </inertial>
-    <!--
-    <inertial>
-      <origin xyz="-9.249840190324093e-15 -6.214898224181922e-17 0.06379502131016988" rpy="0 0 0"/>
-      <mass value="6.892663227665913"/>
-      <inertia ixx="0.021567" iyy="0.021081" izz="0.022375" ixy="0.0" iyz="0.0" ixz="-0.0"/>
-    </inertial>
-    -->
     <visual>
       <origin xyz="0 0 0" rpy="0 0 0"/>
@@ -277,83 +270,3 @@
     </collision>
   </link>
-  <!-- <link name="fl_foot_sphere">
-    <inertial>
-      <origin xyz="0 0 0" rpy="0 0 0"/>
-      <mass value="0.01"/>
-      <inertia ixx="1e-6" iyy="1e-6" izz="1e-6" ixy="0" ixz="0" iyz="0"/>
-    </inertial>
-    <visual>
-      <origin xyz="0 0 0" rpy="0 0 0"/>
-      <geometry>
-        <sphere radius="0.015"/>
-      </geometry>
-      <material name="gray"/>
-    </visual>
-    <collision>
-      <origin xyz="0 0 0" rpy="0 0 0"/>
-      <geometry>
-        <sphere radius="0.015"/>
-      </geometry>
-    </collision>
-  </link>
-  <link name="fr_foot_sphere">
-    <inertial>
-      <origin xyz="0 0 0" rpy="0 0 0"/>
-      <mass value="0.01"/>
-      <inertia ixx="1e-6" iyy="1e-6" izz="1e-6" ixy="0" ixz="0" iyz="0"/>
-    </inertial>
-    <visual>
-      <origin xyz="0 0 0" rpy="0 0 0"/>
-      <geometry>
-        <sphere radius="0.015"/>
-      </geometry>
-      <material name="gray"/>
-    </visual>
-    <collision>
-      <origin xyz="0 0 0" rpy="0 0 0"/>
-      <geometry>
-        <sphere radius="0.015"/>
-      </geometry>
-    </collision>
-  </link>
-  <link name="rl_foot_sphere">
-    <inertial>
-      <origin xyz="0 0 0" rpy="0 0 0"/>
-      <mass value="0.01"/>
-      <inertia ixx="1e-6" iyy="1e-6" izz="1e-6" ixy="0" ixz="0" iyz="0"/>
-    </inertial>
-    <visual>
-      <origin xyz="0 0 0" rpy="0 0 0"/>
-      <geometry>
-        <sphere radius="0.015"/>
-      </geometry>
-      <material name="gray"/>
-    </visual>
-    <collision>
-      <origin xyz="0 0 0" rpy="0 0 0"/>
-      <geometry>
-        <sphere radius="0.015"/>
-      </geometry>
-    </collision>
-  </link>
-  <link name="rr_foot_sphere">
-    <inertial>
-      <origin xyz="0 0 0" rpy="0 0 0"/>
-      <mass value="0.01"/>
-      <inertia ixx="1e-6" iyy="1e-6" izz="1e-6" ixy="0" ixz="0" iyz="0"/>
-    </inertial>
-    <visual>
-      <origin xyz="0 0 0" rpy="0 0 0"/>
-      <geometry>
-        <sphere radius="0.015"/>
-      </geometry>
-      <material name="gray"/>
-    </visual>
-    <collision>
-      <origin xyz="0 0 0" rpy="0 0 0"/>
-      <geometry>
-        <sphere radius="0.015"/>
-      </geometry>
-    </collision>
-  </link> -->
 </robot>
