Commit message: add gazebo imu

File: kaqu_gazebo_sim/description/kaqu.urdf.xacro (robot description, xacro)
@@ -6,3 +6,5 @@
     <xacro:include filename="kaqu.trans" />
     <xacro:include filename="kaqu.gazebo" />
+    <xacro:include filename="kaqu_imu.xacro"/>
+    <xacro:imu_sensor_xacro/>
 </robot>

File: kaqu_gazebo_sim/description/kaqu_imu.xacro (robot description, xacro)
@@ -1,36 +1,13 @@
 <?xml version="1.0"?>
 <robot xmlns:xacro="http://ros.org/wiki/xacro">
-  <xacro:macro name="imu_gazebo_plugin" params="parent imu_link topic">
-    <link name="${imu_link}">
-      <inertial>
-        <mass value="0.001"/>
-        <origin xyz="0 0 0"/>
-        <inertia ixx="1e-6" iyy="1e-6" izz="1e-6"
-                 ixy="0.0" ixz="0.0" iyz="0.0"/>
-      </inertial>
-    </link>
-    <joint name="imu_joint" type="fixed">
-      <parent link="${parent}"/>
-      <child link="${imu_link}"/>
-      <origin xyz="0 0 0" rpy="0 0 0"/>
-    </joint>
-    <gazebo reference="${parent}">
-      <gravity>true</gravity>
-      <sensor name="imu_sensor" type="imu">
+  <xacro:macro name="imu_sensor_xacro" params="">
+    <gazebo reference="base_link">
+      <sensor name="kaqu_imu_sensor" type="imu">
+        <pose>0 0 0.02 0 0 0</pose>
         <always_on>true</always_on>
-        <update_rate>100</update_rate>
-        <visualize>true</visualize>
-        <topic>__default_topic__</topic>
-        <plugin filename="libgazebo_ros_imu_sensor.so" name="imu_plugin">
-          <topicName>${topic}</topicName>
-          <bodyName>${imu_link}</bodyName>
-          <updateRateHZ>15.0</updateRateHZ>
-          <gaussianNoise>0.0</gaussianNoise>
-          <xyzOffset>0 0 0</xyzOffset>
-          <rpyOffset>0 0 0</rpyOffset>
-          <frameName>${parent}</frameName>
-          <initialOrientationAsReference>false</initialOrientationAsReference>
-        </plugin>
-        <pose>0 0 0 0 0 0</pose>
+        <update_rate>100.0</update_rate>
+        <topic>imu</topic>
+        <imu/>
+         <!--imu 속도, 가속도, 방향-->
       </sensor>
     </gazebo>
