Commit message: Edit Foot Contact (Not Work)

File: kaqu_gazebo_sim/description/kaqu_link.xacro (robot description, xacro)
@@ -277,5 +277,5 @@
         ixx="1.843e-7" ixy="1.843e-7" ixz="1.843e-7" iyy="0.0" iyz="0.0" izz="0.0"/>
     </inertial>
-    <collision>
+    <collision name="fl_foot_collision">
       <origin xyz="0 0 0" rpy="0 0 0"/>
       <geometry>
@@ -291,5 +291,5 @@
         ixx="1.843e-7" ixy="1.843e-7" ixz="1.843e-7" iyy="0.0" iyz="0.0" izz="0.0"/>
     </inertial>
-    <collision>
+    <collision name="rl_foot_collision">
       <origin xyz="0 0 0" rpy="0 0 0"/>
       <geometry>
@@ -305,5 +305,5 @@
         ixx="1.843e-7" ixy="1.843e-7" ixz="1.843e-7" iyy="0.0" iyz="0.0" izz="0.0"/>
     </inertial>
-    <collision>
+    <collision name="fr_foot_collision">
       <origin xyz="0 0 0" rpy="0 0 0"/>
       <geometry>
@@ -319,5 +319,5 @@
         ixx="1.843e-7" ixy="1.843e-7" ixz="1.843e-7" iyy="0.0" iyz="0.0" izz="0.0"/>
     </inertial>
-    <collision>
+    <collision name="rr_foot_collision">
       <origin xyz="0 0 0" rpy="0 0 0"/>
       <geometry>

File: kaqu_gazebo_sim/description/sensors/kaqu_contact_feet.xacro (robot description, xacro)
@@ -2,7 +2,4 @@
 <robot xmlns:xacro="http://www.ros.org/wiki/xacro" name="contact_feet_sensors">
   <gazebo reference="fl_foot">
-    <!-- Contact 시스템 플러그인 -->
-    <plugin filename="libignition-gazebo-contact-system.so"
-            name="ignition::gazebo::systems::Contact"/>
     <!-- Contact 센서 -->
     <sensor name="fl_foot_contact" type="contact">
@@ -10,38 +7,38 @@
       <update_rate>200</update_rate>
       <contact>
-        <collision>collision</collision> <!-- 해당 링크 안 collision 이름 -->
+        <collision>fl_foot_collision</collision> <!-- 해당 링크 안 collision 이름 -->
       </contact>
     </sensor>
+    <plugin filename="libignition-gazebo-touchplugin-system.so"
+          name="ignition::gazebo::systems::TouchPlugin">
+      <namespace>fl_foot</namespace>
+      <time>0.001</time>
+      <enabled>true</enabled>
+    </plugin>
   </gazebo>
   <gazebo reference="fr_foot">
-    <plugin filename="libignition-gazebo-contact-system.so"
-            name="ignition::gazebo::systems::Contact"/>
     <sensor name="fr_foot_contact" type="contact">
       <always_on>true</always_on>
       <update_rate>200</update_rate>
       <contact>
-        <collision>collision</collision>
+        <collision>fr_foot_collision</collision>
       </contact>
     </sensor>
   </gazebo>
   <gazebo reference="rl_foot">
-    <plugin filename="libignition-gazebo-contact-system.so"
-            name="ignition::gazebo::systems::Contact"/>
     <sensor name="rl_foot_contact" type="contact">
       <always_on>true</always_on>
       <update_rate>200</update_rate>
       <contact>
-        <collision>collision</collision>
+        <collision>rl_foot_collision</collision>
       </contact>
     </sensor>
   </gazebo>
   <gazebo reference="rr_foot">
-    <plugin filename="libignition-gazebo-contact-system.so"
-            name="ignition::gazebo::systems::Contact"/>
     <sensor name="rr_foot_contact" type="contact">
       <always_on>true</always_on>
       <update_rate>200</update_rate>
       <contact>
-        <collision>collision</collision>
+        <collision>rr_foot_collision</collision>
       </contact>
     </sensor>

Commit message: Update kaqu_link.xacro

File: kaqu_gazebo_sim/description/kaqu_link.xacro (robot description, xacro)
@@ -201,7 +201,13 @@
     </visual>
     <collision>
-      <origin xyz="-0.007 0.05 0.0" rpy="-1.5708 0 0"/>
-      <geometry>
-        <cylinder radius="0.01" length="0.10"/>
+      <origin xyz="-0.007 0.05 0.002" rpy="-1.5708 0 0"/>
+      <geometry>
+        <cylinder radius="0.01" length="0.10"/>
+      </geometry>
+    </collision>
+    <collision>
+      <origin xyz="-0.007 0.102 0.002" rpy="0 0 0"/>
+      <geometry>
+        <sphere radius="0.01"/>
       </geometry>
     </collision>
@@ -222,7 +228,13 @@
     </visual>
     <collision>
-      <origin xyz="-0.007 0.05 0.0" rpy="-1.5708 0 0"/>
-      <geometry>
-        <cylinder radius="0.01" length="0.10"/>
+      <origin xyz="-0.007 0.05 0.002" rpy="-1.5708 0 0"/>
+      <geometry>
+        <cylinder radius="0.01" length="0.10"/>
+      </geometry>
+    </collision>
+      <collision>
+      <origin xyz="-0.007 0.102 0.002" rpy="0 0 0"/>
+      <geometry>
+        <sphere radius="0.01"/>
       </geometry>
     </collision>
@@ -243,7 +255,13 @@
     </visual>
     <collision>
-      <origin xyz="0.007 0.05 0.0" rpy="-1.5708 0 0"/>
-      <geometry>
-        <cylinder radius="0.01" length="0.10"/>
+      <origin xyz="0.007 0.05 0.002" rpy="-1.5708 0 0"/>
+      <geometry>
+        <cylinder radius="0.01" length="0.10"/>
+      </geometry>
+    </collision>
+    <collision>
+      <origin xyz="0.007 0.102 0.002" rpy="0 0 0"/>
+      <geometry>
+        <sphere radius="0.01"/>
       </geometry>
     </collision>
@@ -264,61 +282,11 @@
     </visual>
     <collision>
-      <origin xyz="0.007 0.05 0.0" rpy="-1.5708 0 0"/>
-      <geometry>
-        <cylinder radius="0.01" length="0.10"/>
-      </geometry>
-    </collision>
-  </link>
-  <link name="fl_foot">
-    <inertial>
-      <origin xyz="0 0 0" rpy="0 0 0"/>
-      <mass value="0.0046"/>
-      <inertia
-        ixx="1.843e-7" ixy="1.843e-7" ixz="1.843e-7" iyy="0.0" iyz="0.0" izz="0.0"/>
-    </inertial>
-    <collision>
-      <origin xyz="0 0 0" rpy="0 0 0"/>
-      <geometry>
-        <sphere radius="0.01"/>
-      </geometry>
-    </collision>
-  </link>
-  <link name="rl_foot">
-    <inertial>
-      <origin xyz="0 0 0" rpy="0 0 0"/>
-      <mass value="0.0046"/>
-      <inertia
-        ixx="1.843e-7" ixy="1.843e-7" ixz="1.843e-7" iyy="0.0" iyz="0.0" izz="0.0"/>
-    </inertial>
-    <collision>
-      <origin xyz="0 0 0" rpy="0 0 0"/>
-      <geometry>
-        <sphere radius="0.01"/>
-      </geometry>
-    </collision>
-  </link>
-  <link name="fr_foot">
-    <inertial>
-      <origin xyz="0 0 0" rpy="0 0 0"/>
-      <mass value="0.0046"/>
-      <inertia
-        ixx="1.843e-7" ixy="1.843e-7" ixz="1.843e-7" iyy="0.0" iyz="0.0" izz="0.0"/>
-    </inertial>
-    <collision>
-      <origin xyz="0 0 0" rpy="0 0 0"/>
-      <geometry>
-        <sphere radius="0.01"/>
-      </geometry>
-    </collision>
-  </link>
-  <link name="rr_foot">
-    <inertial>
-      <origin xyz="0 0 0" rpy="0 0 0"/>
-      <mass value="0.0046"/>
-      <inertia
-        ixx="1.843e-7" ixy="1.843e-7" ixz="1.843e-7" iyy="0.0" iyz="0.0" izz="0.0"/>
-    </inertial>
-    <collision>
-      <origin xyz="0 0 0" rpy="0 0 0"/>
+      <origin xyz="0.007 0.05 0.002" rpy="-1.5708 0 0"/>
+      <geometry>
+        <cylinder radius="0.01" length="0.10"/>
+      </geometry>
+    </collision>
+    <collision>
+      <origin xyz="0.007 0.102 0.002" rpy="0 0 0"/>
       <geometry>
         <sphere radius="0.01"/>
