Commit message: CHANGE Effort, Velocity

File: kaqu_gazebo_sim/description/kaqu_joint.xacro (robot description, xacro)
@@ -3,6 +3,7 @@
     <xacro:include filename="$(find kaqu_gazebo_sim)/description/kaqu.gazebo" />
     <xacro:include filename="$(find kaqu_gazebo_sim)/description/kaqu.trans" />
-    <xacro:property name="effort_limit" value="10.0" />
-    <xacro:property name="velocity_limit" value="3.0" />
+    <xacro:property name="effort_limit" value="3.0" />
+    <xacro:property name="velocity_limit" value="10.0" />
+    <!-- 실제 velocity limit: 6내외 -->
     <joint name="fl_mainbodyhip_joint" type="revolute">
         <origin xyz="-0.074 0.077 0.04925" rpy="0 0 0"/>

Commit message: Update kaqu_joint.xacro

File: kaqu_gazebo_sim/description/kaqu_joint.xacro (robot description, xacro)
@@ -3,6 +3,6 @@
     <xacro:include filename="$(find kaqu_gazebo_sim)/description/kaqu.gazebo" />
     <xacro:include filename="$(find kaqu_gazebo_sim)/description/kaqu.trans" />
-    <xacro:property name="effort_limit" value="10.0" />
-    <xacro:property name="velocity_limit" value="3.0" />
+    <xacro:property name="effort_limit" value="3.0" />
+    <xacro:property name="velocity_limit" value="8.0" />
     <joint name="fl_mainbodyhip_joint" type="revolute">
         <origin xyz="-0.074 0.077 0.04925" rpy="0 0 0"/>

Commit message: Edit Collision

File: kaqu_gazebo_sim/description/kaqu_joint.xacro (robot description, xacro)
@@ -3,5 +3,5 @@
     <xacro:include filename="$(find kaqu_gazebo_sim)/description/kaqu.gazebo" />
     <xacro:include filename="$(find kaqu_gazebo_sim)/description/kaqu.trans" />
-    <xacro:property name="effort_limit" value="20.0" />
+    <xacro:property name="effort_limit" value="10.0" />
     <xacro:property name="velocity_limit" value="10.0" />
     <joint name="fl_mainbodyhip_joint" type="revolute">
@@ -163,23 +163,23 @@
         </ros2_control>
     </joint>
-     <!-- <joint name="fl_foot_sphere_joint" type="fixed">
+     <joint name="fl_foot_joint" type="fixed">
         <parent link="fl_leg4_1"/>
-        <child link="fl_foot_sphere"/>
-        <origin xyz="0 0.1 0" rpy="0 0 0"/>
+        <child link="fl_foot"/>
+        <origin xyz="-0.007 0.103 0.002" rpy="0 0 0"/>
      </joint>
-      <joint name="fr_foot_sphere_joint" type="fixed">
+      <joint name="fr_foot_joint" type="fixed">
         <parent link="fr_leg4_1"/>
-        <child link="fr_foot_sphere"/>
-        <origin xyz="0 0.1 0" rpy="0 0 0"/>
+        <child link="fr_foot"/>
+        <origin xyz="0.007 0.103 0.002" rpy="0 0 0"/>
      </joint>
-      <joint name="rl_foot_sphere_joint" type="fixed">
+      <joint name="rl_foot_joint" type="fixed">
         <parent link="rl_leg4_1"/>
-        <child link="rl_foot_sphere"/>
-        <origin xyz="0 0.1 0" rpy="0 0 0"/>
+        <child link="rl_foot"/>
+        <origin xyz="-0.007 0.103 0.002" rpy="0 0 0"/>
      </joint>
-      <joint name="rr_foot_sphere_joint" type="fixed">
+      <joint name="rr_foot_joint" type="fixed">
         <parent link="rr_leg4_1"/>
-        <child link="rr_foot_sphere"/>
-        <origin xyz="0 0.1 0" rpy="0 0 0"/>
-     </joint> -->
+        <child link="rr_foot"/>
+        <origin xyz="0.007 0.103 0.002" rpy="0 0 0"/>
+     </joint>
 </robot>

File: kaqu_gazebo_sim/description/kaqu_link.xacro (robot description, xacro)
@@ -20,7 +20,7 @@
     </visual>
     <collision>
-      <origin xyz="0 0 0" rpy="0 0 0"/>
-      <geometry>
-        <mesh filename="file://$(find kaqu_gazebo_sim)/description/meshes/base_link.stl" scale="0.001 0.001 0.001"/>
+      <origin xyz="0 0 0.05" rpy="0 0 0"/>
+      <geometry>
+        <box size="0.14 0.20 0.05"/>
       </geometry>
     </collision>
@@ -40,7 +40,7 @@
     </visual>
     <collision>
-      <origin xyz="0.074 -0.077 -0.04925" rpy="0 0 0"/>
-      <geometry>
-        <mesh filename="file://$(find kaqu_gazebo_sim)/description/meshes/fl_hip_1.stl" scale="0.001 0.001 0.001"/>
+      <origin xyz="0.0 0.03 -0.0" rpy="0 0 0"/>
+      <geometry>
+        <box size="0.04 0.05 0.065"/>
       </geometry>
     </collision>
@@ -60,7 +60,7 @@
     </visual>
     <collision>
-      <origin xyz="-0.074 -0.077 -0.04925" rpy="0 0 0"/>
-      <geometry>
-        <mesh filename="file://$(find kaqu_gazebo_sim)/description/meshes/fr_hip_1.stl" scale="0.001 0.001 0.001"/>
+      <origin xyz="0.0 0.03 -0.0" rpy="0 0 0"/>
+      <geometry>
+        <box size="0.04 0.05 0.065"/>
       </geometry>
     </collision>
@@ -80,7 +80,7 @@
     </visual>
     <collision>
-      <origin xyz="0.074 0.077 -0.04925" rpy="0 0 0"/>
-      <geometry>
-        <mesh filename="file://$(find kaqu_gazebo_sim)/description/meshes/rl_hip_1.stl" scale="0.001 0.001 0.001"/>
+      <origin xyz="0.0 -0.03 -0.0" rpy="0 0 0"/>
+      <geometry>
+        <box size="0.04 0.05 0.065"/>
       </geometry>
     </collision>
@@ -100,7 +100,7 @@
     </visual>
     <collision>
-      <origin xyz="-0.074 0.077 -0.04925" rpy="0 0 0"/>
-      <geometry>
-        <mesh filename="file://$(find kaqu_gazebo_sim)/description/meshes/rr_hip_1.stl" scale="0.001 0.001 0.001"/>
+      <origin xyz="0.0 -0.03 -0.0" rpy="0 0 0"/>
+      <geometry>
+        <box size="0.04 0.05 0.065"/>
       </geometry>
     </collision>
@@ -120,7 +120,7 @@
     </visual>
     <collision>
-      <origin xyz="0.095 -0.11625 -0.0335" rpy="0 0 0"/>
-      <geometry>
-        <mesh filename="file://$(find kaqu_gazebo_sim)/description/meshes/fl_leg1_1.stl" scale="0.001 0.001 0.001"/>
+      <origin xyz="-0.02 -0.05 0.0" rpy="-1.5708 0 0"/>
+      <geometry>
+        <cylinder radius="0.015" length="0.10"/>
       </geometry>
     </collision>
@@ -140,7 +140,7 @@
     </visual>
     <collision>
-      <origin xyz="0.095 0.09225 -0.0335" rpy="0 0 0"/>
-      <geometry>
-        <mesh filename="file://$(find kaqu_gazebo_sim)/description/meshes/rl_leg1_1.stl" scale="0.001 0.001 0.001"/>
+      <origin xyz="-0.02 -0.05 0.0" rpy="-1.5708 0 0"/>
+      <geometry>
+        <cylinder radius="0.015" length="0.10"/>
       </geometry>
     </collision>
@@ -160,7 +160,7 @@
     </visual>
     <collision>
-      <origin xyz="-0.095 -0.11625 -0.0335" rpy="0 0 0"/>
-      <geometry>
-        <mesh filename="file://$(find kaqu_gazebo_sim)/description/meshes/fr_leg1_1.stl" scale="0.001 0.001 0.001"/>
+      <origin xyz="0.02 -0.05 0.0" rpy="-1.5708 0 0"/>
+      <geometry>
+        <cylinder radius="0.015" length="0.10"/>
       </geometry>
     </collision>
@@ -180,7 +180,7 @@
     </visual>
     <collision>
-      <origin xyz="-0.095 0.09225 -0.0335" rpy="0 0 0"/>
-      <geometry>
-        <mesh filename="file://$(find kaqu_gazebo_sim)/description/meshes/rr_leg1_1.stl" scale="0.001 0.001 0.001"/>
+      <origin xyz="0.02 -0.05 0.0" rpy="-1.5708 0 0"/>
+      <geometry>
+        <cylinder radius="0.015" length="0.10"/>
       </geometry>
     </collision>
@@ -201,7 +201,7 @@
     </visual>
     <collision>
-      <origin xyz="0.107 -0.01625 -0.0335" rpy="0 0 0"/>
-      <geometry>
-        <mesh filename="file://$(find kaqu_gazebo_sim)/description/meshes/fl_leg4_1_0.stl" scale="0.001 0.001 0.001"/>
+      <origin xyz="-0.007 0.05 0.0" rpy="-1.5708 0 0"/>
+      <geometry>
+        <cylinder radius="0.01" length="0.10"/>
       </geometry>
     </collision>
@@ -222,7 +222,7 @@
     </visual>
     <collision>
-      <origin xyz="0.107 0.19225 -0.0335" rpy="0 0 0"/>
-      <geometry>
-        <mesh filename="file://$(find kaqu_gazebo_sim)/description/meshes/rl_leg4_1_0.stl" scale="0.001 0.001 0.001"/>
+      <origin xyz="-0.007 0.05 0.0" rpy="-1.5708 0 0"/>
+      <geometry>
+        <cylinder radius="0.01" length="0.10"/>
       </geometry>
     </collision>
@@ -243,7 +243,7 @@
     </visual>
     <collision>
-      <origin xyz="-0.107 -0.01625 -0.0335" rpy="0 0 0"/>
-      <geometry>
-        <mesh filename="file://$(find kaqu_gazebo_sim)/description/meshes/fr_leg4_1_0.stl" scale="0.001 0.001 0.001"/>
+      <origin xyz="0.007 0.05 0.0" rpy="-1.5708 0 0"/>
+      <geometry>
+        <cylinder radius="0.01" length="0.10"/>
       </geometry>
     </collision>
@@ -264,7 +264,63 @@
     </visual>
     <collision>
-      <origin xyz="-0.107 0.19225 -0.0335" rpy="0 0 0"/>
-      <geometry>
-        <mesh filename="file://$(find kaqu_gazebo_sim)/description/meshes/rr_leg4_1_0.stl" scale="0.001 0.001 0.001"/>
+      <origin xyz="0.007 0.05 0.0" rpy="-1.5708 0 0"/>
+      <geometry>
+        <cylinder radius="0.01" length="0.10"/>
+      </geometry>
+    </collision>
+  </link>
+  <link name="fl_foot">
+    <inertial>
+      <origin xyz="0 0 0" rpy="0 0 0"/>
+      <mass value="0.0046"/>
+      <inertia
+        ixx="1.843e-7" ixy="1.843e-7" ixz="1.843e-7" iyy="0.0" iyz="0.0" izz="0.0"/>
+    </inertial>
+    <collision>
+      <origin xyz="0 0 0" rpy="0 0 0"/>
+      <geometry>
+        <sphere radius="0.01"/>
+      </geometry>
+    </collision>
+  </link>
+  <link name="rl_foot">
+    <inertial>
+      <origin xyz="0 0 0" rpy="0 0 0"/>
+      <mass value="0.0046"/>
+      <inertia
+        ixx="1.843e-7" ixy="1.843e-7" ixz="1.843e-7" iyy="0.0" iyz="0.0" izz="0.0"/>
+    </inertial>
+    <collision>
+      <origin xyz="0 0 0" rpy="0 0 0"/>
+      <geometry>
+        <sphere radius="0.01"/>
+      </geometry>
+    </collision>
+  </link>
+  <link name="fr_foot">
+    <inertial>
+      <origin xyz="0 0 0" rpy="0 0 0"/>
+      <mass value="0.0046"/>
+      <inertia
+        ixx="1.843e-7" ixy="1.843e-7" ixz="1.843e-7" iyy="0.0" iyz="0.0" izz="0.0"/>
+    </inertial>
+    <collision>
+      <origin xyz="0 0 0" rpy="0 0 0"/>
+      <geometry>
+        <sphere radius="0.01"/>
+      </geometry>
+    </collision>
+  </link>
+  <link name="rr_foot">
+    <inertial>
+      <origin xyz="0 0 0" rpy="0 0 0"/>
+      <mass value="0.0046"/>
+      <inertia
+        ixx="1.843e-7" ixy="1.843e-7" ixz="1.843e-7" iyy="0.0" iyz="0.0" izz="0.0"/>
+    </inertial>
+    <collision>
+      <origin xyz="0 0 0" rpy="0 0 0"/>
+      <geometry>
+        <sphere radius="0.01"/>
       </geometry>
     </collision>

Commit message: Add Contact Sensor (Work)

File: kaqu_gazebo_sim/description/kaqu_joint.xacro (robot description, xacro)
@@ -163,23 +163,3 @@
         </ros2_control>
     </joint>
-     <joint name="fl_foot_joint" type="fixed">
-        <parent link="fl_leg4_1"/>
-        <child link="fl_foot"/>
-        <origin xyz="-0.007 0.103 0.002" rpy="0 0 0"/>
-     </joint>
-      <joint name="fr_foot_joint" type="fixed">
-        <parent link="fr_leg4_1"/>
-        <child link="fr_foot"/>
-        <origin xyz="0.007 0.103 0.002" rpy="0 0 0"/>
-     </joint>
-      <joint name="rl_foot_joint" type="fixed">
-        <parent link="rl_leg4_1"/>
-        <child link="rl_foot"/>
-        <origin xyz="-0.007 0.103 0.002" rpy="0 0 0"/>
-     </joint>
-      <joint name="rr_foot_joint" type="fixed">
-        <parent link="rr_leg4_1"/>
-        <child link="rr_foot"/>
-        <origin xyz="0.007 0.103 0.002" rpy="0 0 0"/>
-     </joint>
 </robot>

File: kaqu_gazebo_sim/description/kaqu_link.xacro (robot description, xacro)
@@ -201,7 +201,13 @@
     </visual>
     <collision>
-      <origin xyz="-0.007 0.05 0.0" rpy="-1.5708 0 0"/>
-      <geometry>
-        <cylinder radius="0.01" length="0.10"/>
+      <origin xyz="-0.007 0.05 0.002" rpy="-1.5708 0 0"/>
+      <geometry>
+        <cylinder radius="0.01" length="0.10"/>
+      </geometry>
+    </collision>
+    <collision>
+      <origin xyz="-0.007 0.102 0.002" rpy="0 0 0"/>
+      <geometry>
+        <sphere radius="0.01"/>
       </geometry>
     </collision>
@@ -222,7 +228,13 @@
     </visual>
     <collision>
-      <origin xyz="-0.007 0.05 0.0" rpy="-1.5708 0 0"/>
-      <geometry>
-        <cylinder radius="0.01" length="0.10"/>
+      <origin xyz="-0.007 0.05 0.002" rpy="-1.5708 0 0"/>
+      <geometry>
+        <cylinder radius="0.01" length="0.10"/>
+      </geometry>
+    </collision>
+      <collision>
+      <origin xyz="-0.007 0.102 0.002" rpy="0 0 0"/>
+      <geometry>
+        <sphere radius="0.01"/>
       </geometry>
     </collision>
@@ -243,7 +255,13 @@
     </visual>
     <collision>
-      <origin xyz="0.007 0.05 0.0" rpy="-1.5708 0 0"/>
-      <geometry>
-        <cylinder radius="0.01" length="0.10"/>
+      <origin xyz="0.007 0.05 0.002" rpy="-1.5708 0 0"/>
+      <geometry>
+        <cylinder radius="0.01" length="0.10"/>
+      </geometry>
+    </collision>
+    <collision>
+      <origin xyz="0.007 0.102 0.002" rpy="0 0 0"/>
+      <geometry>
+        <sphere radius="0.01"/>
       </geometry>
     </collision>
@@ -264,61 +282,11 @@
     </visual>
     <collision>
-      <origin xyz="0.007 0.05 0.0" rpy="-1.5708 0 0"/>
-      <geometry>
-        <cylinder radius="0.01" length="0.10"/>
-      </geometry>
-    </collision>
-  </link>
-  <link name="fl_foot">
-    <inertial>
-      <origin xyz="0 0 0" rpy="0 0 0"/>
-      <mass value="0.0046"/>
-      <inertia
-        ixx="1.843e-7" ixy="1.843e-7" ixz="1.843e-7" iyy="0.0" iyz="0.0" izz="0.0"/>
-    </inertial>
-    <collision name="fl_foot_collision">
-      <origin xyz="0 0 0" rpy="0 0 0"/>
-      <geometry>
-        <sphere radius="0.01"/>
-      </geometry>
-    </collision>
-  </link>
-  <link name="rl_foot">
-    <inertial>
-      <origin xyz="0 0 0" rpy="0 0 0"/>
-      <mass value="0.0046"/>
-      <inertia
-        ixx="1.843e-7" ixy="1.843e-7" ixz="1.843e-7" iyy="0.0" iyz="0.0" izz="0.0"/>
-    </inertial>
-    <collision name="rl_foot_collision">
-      <origin xyz="0 0 0" rpy="0 0 0"/>
-      <geometry>
-        <sphere radius="0.01"/>
-      </geometry>
-    </collision>
-  </link>
-  <link name="fr_foot">
-    <inertial>
-      <origin xyz="0 0 0" rpy="0 0 0"/>
-      <mass value="0.0046"/>
-      <inertia
-        ixx="1.843e-7" ixy="1.843e-7" ixz="1.843e-7" iyy="0.0" iyz="0.0" izz="0.0"/>
-    </inertial>
-    <collision name="fr_foot_collision">
-      <origin xyz="0 0 0" rpy="0 0 0"/>
-      <geometry>
-        <sphere radius="0.01"/>
-      </geometry>
-    </collision>
-  </link>
-  <link name="rr_foot">
-    <inertial>
-      <origin xyz="0 0 0" rpy="0 0 0"/>
-      <mass value="0.0046"/>
-      <inertia
-        ixx="1.843e-7" ixy="1.843e-7" ixz="1.843e-7" iyy="0.0" iyz="0.0" izz="0.0"/>
-    </inertial>
-    <collision name="rr_foot_collision">
-      <origin xyz="0 0 0" rpy="0 0 0"/>
+      <origin xyz="0.007 0.05 0.002" rpy="-1.5708 0 0"/>
+      <geometry>
+        <cylinder radius="0.01" length="0.10"/>
+      </geometry>
+    </collision>
+    <collision>
+      <origin xyz="0.007 0.102 0.002" rpy="0 0 0"/>
       <geometry>
         <sphere radius="0.01"/>

File: kaqu_gazebo_sim/description/sensors/kaqu_contact_feet.xacro (robot description, xacro)
@@ -1,5 +1,5 @@
 <?xml version="1.0"?>
 <robot xmlns:xacro="http://www.ros.org/wiki/xacro" name="contact_feet_sensors">
-  <gazebo reference="fl_foot">
+  <gazebo reference="fl_leg4_1">
     <!-- Contact 센서 -->
     <sensor name="fl_foot_contact" type="contact">
@@ -7,5 +7,6 @@
       <update_rate>200</update_rate>
       <contact>
-        <collision>fl_foot_collision</collision> <!-- 해당 링크 안 collision 이름 -->
+      <!-- 가제보 시뮬레이션상에서 기본 collision 이름 -->
+        <collision>fl_leg4_1_collision_1</collision> <!-- 해당 링크 안 collision 이름 -->
       </contact>
     </sensor>
@@ -17,28 +18,28 @@
     </plugin>
   </gazebo>
-  <gazebo reference="fr_foot">
+  <gazebo reference="fr_leg4_1">
     <sensor name="fr_foot_contact" type="contact">
       <always_on>true</always_on>
       <update_rate>200</update_rate>
       <contact>
-        <collision>fr_foot_collision</collision>
+        <collision>fr_leg4_1_collision_1</collision>
       </contact>
     </sensor>
   </gazebo>
-  <gazebo reference="rl_foot">
+  <gazebo reference="rl_leg4_1">
     <sensor name="rl_foot_contact" type="contact">
       <always_on>true</always_on>
       <update_rate>200</update_rate>
       <contact>
-        <collision>rl_foot_collision</collision>
+        <collision>rl_leg4_1_collision_1</collision>
       </contact>
     </sensor>
   </gazebo>
-  <gazebo reference="rr_foot">
+  <gazebo reference="rr_leg4_1">
     <sensor name="rr_foot_contact" type="contact">
       <always_on>true</always_on>
       <update_rate>200</update_rate>
       <contact>
-        <collision>rr_foot_collision</collision>
+        <collision>rr_leg4_1_collision_1</collision>
       </contact>
     </sensor>

Commit message: Edit effort, Velocity

File: kaqu_gazebo_sim/description/kaqu_joint.xacro (robot description, xacro)
@@ -3,6 +3,6 @@
     <xacro:include filename="$(find kaqu_gazebo_sim)/description/kaqu.gazebo" />
     <xacro:include filename="$(find kaqu_gazebo_sim)/description/kaqu.trans" />
-    <xacro:property name="effort_limit" value="10.0" />
-    <xacro:property name="velocity_limit" value="10.0" />
+    <xacro:property name="effort_limit" value="4.0" />
+    <xacro:property name="velocity_limit" value="6.0" />
     <joint name="fl_mainbodyhip_joint" type="revolute">
         <origin xyz="-0.074 0.077 0.04925" rpy="0 0 0"/>
